File: SC - Matrix Board/SC - Matrix Board.kicad_pcb (KiCad board)
At the start: 2 copper layers, 126 x 83.3 mm, 120 parts, among them J2 Conn_01x09_Pin

Commit message: updated after first CL DR
Routing:
- net /E_1: track 33.3 -> 36.2 mm
- net /E_button: track 51.1 -> 52.9 mm
- net /E_2: track 33.7 -> 35.2 mm
Changed lines of the file:
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@@
 	)
 	(segment
-		(start 114.286618 62.686618)
-		(end 113.8 63.173236)
-		(width 0.5)
-		(layer "F.Cu")
-		(net 1)
-	)
-	(segment
 		(start 86.36 83.2)
 		(end 87.6 83.2)
@@
 	)
 	(segment
+		(start 123.72 66.8)
+		(end 123 66.8)
+		(width 0.5)
+		(layer "F.Cu")
+		(net 1)
+	)
+	(segment
+		(start 113.88 63.8)
+		(end 113.8 63.72)
+		(width 0.5)
+		(layer "F.Cu")
+		(net 1)
+	)
+	(segment
 		(start 68.924707 57.924707)
 		(end 66.6 55.6)
@@
 	)
 	(segment
+		(start 115 63.8)
+		(end 113.88 63.8)
+		(width 0.5)
+		(layer "F.Cu")
+		(net 1)
+	)
+	(segment
 		(start 80.35 83.4)
 		(end 79.28 83.4)
@@
 	)
 	(segment
+		(start 123 66.8)
+		(end 122.6 66.4)
+		(width 0.5)
+		(layer "F.Cu")
+		(net 1)
+	)
+	(segment
 		(start 133.624073 59.48162)
 		(end 130.2 56.057547)
@@
 	)
 	(segment
-		(start 123.72 66.8)
-		(end 122.6 66.8)
-		(width 0.5)
-		(layer "F.Cu")
-		(net 1)
-	)
-	(segment
 		(start 81.6 94.64878)
 		(end 83.062086 94.64878)
@@
 	)
 	(segment
-		(start 113.8 63.173236)
-		(end 113.8 63.72)
-		(width 0.5)
-		(layer "F.Cu")
-		(net 1)
-	)
-	(segment
 		(start 61.2 70.031161)
 		(end 59.612964 70.031161)
@@
 	)
 	(via
-		(at 122.6 66.8)
+		(at 122.6 66.4)
 		(size 0.6)
 		(drill 0.3)
@@
 	)
 	(via
-		(at 114.286618 62.686618)
+		(at 115 63.8)
 		(size 0.6)
 		(drill 0.3)
@@
 	(segment
 		(start 87 68.2)
-		(end 89.2 70.4)
+		(end 91 72.2)
 		(width 0.2)
 		(layer "B.Cu")
@@
 	)
 	(segment
-		(start 89.2 70.4)
-		(end 105.724707 70.4)
+		(start 91 72.2)
+		(end 103.924707 72.2)
 		(width 0.2)
 		(layer "B.Cu")
@@
 	)
 	(segment
-		(start 105.724707 70.4)
+		(start 103.924707 72.2)
 		(end 115.7 60.424707)
 		(width 0.2)
@@
 	)
 	(segment
-		(start 88.2 71.4)
-		(end 119.224707 71.4)
+		(start 90.4 73.6)
+		(end 117.024707 73.6)
 		(width 0.2)
 		(layer "B.Cu")
@@
 	(segment
 		(start 85 68.2)
-		(end 88.2 71.4)
+		(end 90.4 73.6)
 		(width 0.2)
 		(layer "B.Cu")
@@
 	)
 	(segment
-		(start 119.224707 71.4)
+		(start 117.024707 73.6)
 		(end 130.2 60.424707)
 		(width 0.2)
@@
 	)
 	(segment
-		(start 101.324707 69.8)
-		(end 115.7 55.424707)
+		(start 89 68.2)
+		(end 91.8 71)
 		(width 0.2)
 		(layer "B.Cu")
@@
 	)
 	(segment
-		(start 89 68.2)
-		(end 90.6 69.8)
+		(start 111.8 62.6)
+		(end 111.8 59.324707)
+		(width 0.2)
+		(layer "B.Cu")
+		(net 61)
+	)
+	(segment
+		(start 103.4 71)
+		(end 111.8 62.6)
+		(width 0.2)
+		(layer "B.Cu")
+		(net 61)
+	)
+	(segment
+		(start 111.8 59.324707)
+		(end 115.7 55.424707)
 		(width 0.2)
 		(layer "B.Cu")
@@
 	)
 	(segment
-		(start 90.6 69.8)
-		(end 101.324707 69.8)
+		(start 91.8 71)
+		(end 103.4 71)
 		(width 0.2)
 		(layer "B.Cu")
