File: SC - Teensy Board/SC - Teensy Board.kicad_pcb (KiCad board)
At the start: 2 copper layers, 40.5 x 90 mm, 14 parts, among them J1 Conn_01x15_Pin, J2 Conn_01x02_Pin, J3 Conn_01x24_Socket, J4 Conn_01x24_Socket, J5 Conn_01x06_Pin, J6 Conn_01x03_Pin, J7 Conn_01x03_Pin, U1 Teensy4.1

Commit message: updated after first CL DR
Routing:
- net GND: track 19.5 -> 0.00 mm, vias 7 -> 0
Changed lines of the file:
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@@
 					(xy 55.955261 42.995987) (xy 55.961367 41.787229) (xy 55.977976 41.552267) (xy 56.039157 41.383393)
 					(xy 56.126409 41.251163) (xy 56.240048 41.149267) (xy 56.256901 41.138032) (xy 56.329197 41.087718)
-					(xy 56.758576 40.925296) (xy 56.758576 39.375332) (xy 56.183887 39.598182) (xy 56.011437 39.683078)
-					(xy 55.977732 39.711166) (xy 55.894109 39.780443) (xy 55.820439 39.867726) (xy 55.747687 40.002391)
-					(xy 55.698566 40.189229) (xy 55.68 40.444138) (xy 55.68 43.376517) (xy 55.699623 43.551125) (xy 55.749123 43.658685)
+					(xy 56.758576 40.925296) (xy 56.758576 39.375331) (xy 56.183887 39.598181) (xy 56.011437 39.683077)
+					(xy 55.977732 39.711165) (xy 55.894109 39.780442) (xy 55.820439 39.867725) (xy 55.747687 40.00239)
+					(xy 55.698566 40.189228) (xy 55.68 40.444138) (xy 55.68 43.376517) (xy 55.699623 43.551125) (xy 55.749123 43.658685)
 					(xy 55.822571 43.720699)
 				)
@@
 			(polygon
 				(pts
-					(xy 58.582093 36.40192) (xy 58.465101 36.440998) (xy 58.345842 36.468804) (xy 58.258051 36.464479)
-					(xy 58.192037 36.435381) (xy 58.146204 36.380805) (xy 58.11364 36.277779) (xy 58.102889 36.099791)
-					(xy 58.102889 34.812631) (xy 58.087862 34.567187) (xy 58.050129 34.406075) (xy 57.997996 34.305537)
-					(xy 57.935094 34.247453) (xy 57.839839 34.219365) (xy 57.828604 34.219365) (xy 57.760249 34.230637)
-					(xy 57.604877 34.280915) (xy 56.116461 34.801396) (xy 55.943049 34.896651) (xy 55.828629 34.999046)
-					(xy 55.747688 35.120715) (xy 55.69766 35.265448) (xy 55.68 35.439358) (xy 55.68 38.371738) (xy 55.699219 38.65776)
-					(xy 55.730802 38.780112) (xy 55.798457 38.875367) (xy 55.876565 38.921762) (xy 55.961856 38.936916)
-					(xy 56.001423 38.936916) (xy 56.112155 38.921675) (xy 56.32822 38.858514) (xy 56.711681 38.724181)
-					(xy 56.711681 37.257991) (xy 56.323824 37.381089) (xy 56.209762 37.397942) (xy 56.120916 37.384878)
-					(xy 56.05216 37.347977) (xy 55.998492 37.286079) (xy 55.948664 37.174197) (xy 55.930104 37.017412)
-					(xy 55.930104 36.950245) (xy 55.946731 36.744777) (xy 55.989661 36.60398) (xy 56.052065 36.510455)
-					(xy 56.132826 36.452234) (xy 57.501807 35.976693) (xy 57.637013 35.961236) (xy 57.726999 36.00185)
-					(xy 57.764477 36.056702) (xy 57.793546 36.165089) (xy 57.805889 36.357223) (xy 57.805889 37.582589)
-					(xy 57.82862 37.905134) (xy 57.881825 38.083045) (xy 57.950725 38.170238) (xy 58.004253 38.195298)
-					(xy 58.067718 38.203943) (xy 58.150989 38.19193) (xy 58.312693 38.14215) (xy 59.705122 37.644139)
-					(xy 59.872184 37.554746) (xy 59.979516 37.466827) (xy 60.060393 37.363116) (xy 60.117159 37.241382)
-					(xy 60.14254 37.12473) (xy 60.150621 37.017412) (xy 60.150621 34.264062) (xy 60.144164 33.881301)
-					(xy 60.133768 33.788521) (xy 60.101904 33.670391) (xy 60.060983 33.598256) (xy 59.973366 33.527813)
-					(xy 59.847759 33.503001) (xy 59.720284 33.519371) (xy 59.517055 33.581403) (xy 59.118939 33.715737)
-					(xy 59.118939 35.153839) (xy 59.33778 35.075681) (xy 59.528585 35.017491) (xy 59.635512 35.002897)
-					(xy 59.735346 35.019594) (xy 59.810596 35.067014) (xy 59.867394 35.148714) (xy 59.904912 35.277181)
-					(xy 59.916147 35.450594) (xy 59.916147 36.653734) (xy 59.707564 36.726518) (xy 59.707564 36.592185)
-					(xy 59.689242 36.396903) (xy 59.640642 36.256351) (xy 59.58788 36.194997) (xy 59.517489 36.157846)
-					(xy 59.42351 36.144488) (xy 59.306161 36.15484) (xy 59.211751 36.183566) (xy 58.582093 36.407537)
+					(xy 58.582093 36.401919) (xy 58.465101 36.440997) (xy 58.345842 36.468803) (xy 58.258051 36.464478)
+					(xy 58.192037 36.43538) (xy 58.146204 36.380804) (xy 58.11364 36.277778) (xy 58.102889 36.09979)
+					(xy 58.102889 34.81263) (xy 58.087862 34.567186) (xy 58.050129 34.406074) (xy 57.997996 34.305536)
+					(xy 57.935094 34.247452) (xy 57.839839 34.219364) (xy 57.828604 34.219364) (xy 57.760249 34.230636)
+					(xy 57.604877 34.280914) (xy 56.116461 34.801395) (xy 55.943049 34.89665) (xy 55.828629 34.999045)
+					(xy 55.747688 35.120714) (xy 55.69766 35.265447) (xy 55.68 35.439357) (xy 55.68 38.371737) (xy 55.699219 38.657759)
+					(xy 55.730802 38.780111) (xy 55.798457 38.875366) (xy 55.876565 38.921761) (xy 55.961856 38.936915)
+					(xy 56.001423 38.936915) (xy 56.112155 38.921674) (xy 56.32822 38.858513) (xy 56.711681 38.72418)
+					(xy 56.711681 37.25799) (xy 56.323824 37.381088) (xy 56.209762 37.397941) (xy 56.120916 37.384877)
+					(xy 56.05216 37.347976) (xy 55.998492 37.286078) (xy 55.948664 37.174196) (xy 55.930104 37.017411)
+					(xy 55.930104 36.950244) (xy 55.946731 36.744776) (xy 55.989661 36.603979) (xy 56.052065 36.510454)
+					(xy 56.132826 36.452233) (xy 57.501807 35.976692) (xy 57.637013 35.961235) (xy 57.726999 36.001849)
+					(xy 57.764477 36.056701) (xy 57.793546 36.165088) (xy 57.805889 36.357222) (xy 57.805889 37.582588)
+					(xy 57.82862 37.905133) (xy 57.881825 38.083044) (xy 57.950725 38.170237) (xy 58.004253 38.195297)
+					(xy 58.067718 38.203942) (xy 58.150989 38.191929) (xy 58.312693 38.142149) (xy 59.705122 37.644138)
+					(xy 59.872184 37.554745) (xy 59.979516 37.466826) (xy 60.060393 37.363115) (xy 60.117159 37.241381)
+					(xy 60.14254 37.124729) (xy 60.150621 37.017411) (xy 60.150621 34.264061) (xy 60.144164 33.8813)
+					(xy 60.133768 33.78852) (xy 60.101904 33.67039) (xy 60.060983 33.598255) (xy 59.973366 33.527812)
+					(xy 59.847759 33.503) (xy 59.720284 33.51937) (xy 59.517055 33.581402) (xy 59.118939 33.715736)
+					(xy 59.118939 35.153838) (xy 59.33778 35.07568) (xy 59.528585 35.01749) (xy 59.635512 35.002896)
+					(xy 59.735346 35.019593) (xy 59.810596 35.067013) (xy 59.867394 35.148713) (xy 59.904912 35.27718)
+					(xy 59.916147 35.450593) (xy 59.916147 36.653733) (xy 59.707564 36.726517) (xy 59.707564 36.592184)
+					(xy 59.689242 36.396902) (xy 59.640642 36.25635) (xy 59.58788 36.194996) (xy 59.517489 36.157845)
+					(xy 59.42351 36.144487) (xy 59.306161 36.154839) (xy 59.211751 36.183565) (xy 58.582093 36.407536)
 				)
 			)
@@
 	)
 	(segment
-		(start 63.6 77.349999)
-		(end 65.67 77.349999)
-		(width 0.5)
-		(layer "F.Cu")
-		(net 15)
-	)
-	(segment
-		(start 48 45.8)
-		(end 48 46.4)
-		(width 0.5)
-		(layer "F.Cu")
-		(net 15)
-	)
-	(segment
-		(start 46.6 47.8)
-		(end 45.4 47.8)
-		(width 0.5)
-		(layer "F.Cu")
-		(net 15)
-	)
-	(segment
-		(start 71 61)
-		(end 69 61)
-		(width 0.5)
-		(layer "F.Cu")
-		(net 15)
-	)
-	(segment
-		(start 65.67 44.329999)
-		(end 65.729999 44.329999)
-		(width 0.5)
-		(layer "F.Cu")
-		(net 15)
-	)
-	(segment
-		(start 48 55.6)
-		(end 46.6 57)
-		(width 0.5)
-		(layer "F.Cu")
-		(net 15)
-	)
-	(segment
-		(start 67.6 46.2)
-		(end 68.2 46.2)
-		(width 0.5)
-		(layer "F.Cu")
-		(net 15)
-	)
-	(segment
-		(start 46.6 57)
-		(end 45.4 57)
-		(width 0.5)
-		(layer "F.Cu")
-		(net 15)
-	)
-	(segment
-		(start 48 55.2)
-		(end 48 55.6)
-		(width 0.5)
-		(layer "F.Cu")
-		(net 15)
-	)
-	(segment
-		(start 65.729999 44.329999)
-		(end 67.6 46.2)
-		(width 0.5)
-		(layer "F.Cu")
-		(net 15)
-	)
-	(segment
-		(start 45.4 42)
-		(end 45.4 40.4)
-		(width 0.5)
-		(layer "F.Cu")
-		(net 15)
-	)
-	(segment
-		(start 50.4 41.8)
-		(end 50.4 39.2)
-		(width 0.5)
-		(layer "F.Cu")
-		(net 15)
-	)
-	(segment
-		(start 48 46.4)
-		(end 46.6 47.8)
-		(width 0.5)
-		(layer "F.Cu")
-		(net 15)
-	)
-	(segment
-		(start 69 61)
-		(end 68.6 60.6)
-		(width 0.5)
-		(layer "F.Cu")
-		(net 15)
-	)
-	(via
-		(at 48 45.8)
-		(size 0.6)
-		(drill 0.3)
-		(layers "F.Cu" "B.Cu")
-		(net 15)
-	)
-	(via
-		(at 48 55.2)
-		(size 0.6)
-		(drill 0.3)
-		(layers "F.Cu" "B.Cu")
-		(net 15)
-	)
-	(via
-		(at 50.4 39.2)
-		(size 0.6)
-		(drill 0.3)
-		(layers "F.Cu" "B.Cu")
-		(net 15)
-	)
-	(via
-		(at 68.2 46.2)
-		(size 0.6)
-		(drill 0.3)
-		(layers "F.Cu" "B.Cu")
-		(net 15)
-	)
-	(via
-		(at 68.6 60.6)
-		(size 0.6)
-		(drill 0.3)
-		(layers "F.Cu" "B.Cu")
-		(net 15)
-	)
-	(via
-		(at 45.4 42)
-		(size 0.6)
-		(drill 0.3)
-		(layers "F.Cu" "B.Cu")
-		(net 15)
-	)
-	(via
-		(at 63.6 77.349999)
-		(size 0.6)
-		(drill 0.3)
-		(layers "F.Cu" "B.Cu")
-		(net 15)
-	)
-	(segment
