File: SC - 6 Layer Knob/SC - 6 Layer Knob.kicad_pcb (KiCad board)
At the start: 2 copper layers, 126 x 90 mm, 113 parts, among them J1 Conn_01x15_Pin, J2 Conn_01x09_Pin

Commit message: moved to fit sheet bounds
Parts:
- moved H8 212.3 mm to (194.8, 59.9)
- moved H9 212.3 mm to (94.0, 59.9)
- moved C1 212.3 mm to (105.4, 69.1)
- moved C11 212.3 mm to (137.8, 74.5)
- moved C12 212.3 mm to (146.8, 96.0)
- moved C13 212.3 mm to (135.4, 90.1)
- moved C14 212.3 mm to (134.0, 83.3)
- moved C15 212.3 mm to (146.4, 69.1)
- moved C18 212.3 mm to (194.2, 71.5)
- moved C19 212.3 mm to (187.4, 69.1)
- moved C2 212.3 mm to (112.2, 72.2)
- moved C20 212.3 mm to (178.6, 74.9)
- moved C22 212.3 mm to (176.4, 90.1)
- moved C23 212.3 mm to (187.8, 96.0)
- moved C24 212.3 mm to (192.2, 89.2)
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